Commit message: Remove unused descriptions

File: description/urdf/handrobot_description.urdf.xacro (robot description, xacro)
@@ -15,24 +15,4 @@
         color="yellow"
     />
-    <joint name="base_joint2" type="fixed">
-        <xacro:insert_block name="origin" />
-        <parent link = "${parent}" />
-        <child link = "two_down" />
-    </joint>
-    <joint name="base_joint3" type="fixed">
-        <xacro:insert_block name="origin" />
-        <parent link = "${parent}" />
-        <child link = "three_down" />
-    </joint>
-    <joint name="base_joint4" type="fixed">
-        <xacro:insert_block name="origin" />
-        <parent link = "${parent}" />
-        <child link = "four_down" />
-    </joint>
-    <joint name="base_joint5" type="fixed">
-        <xacro:insert_block name="origin" />
-        <parent link = "${parent}" />
-        <child link = "five_down" />
-    </joint>
     <!-- Joint 1 -->
     <xacro:create_link
