Commit message: Build success files. Yet to try launch robot..

File: description/ros2_control/handrobot.ros2_control.xacro (robot description, xacro)
@@ -1,8 +1,8 @@
 <?xml version="1.0"?>
 <robot xmlns:xacro="https://www.ros.org/wiki/xacro">
-    <xacro:macro name="handRobot_ros2_control" params="name">
+    <xacro:macro name="handrobot_ros2_control" params="name">
         <ros2_control name="${name}", type="system">
             <hardware>
-                <plugin>handRobot_ros2_control/handRobotSystemPositionHardware</plugin>
+                <plugin>handrobot_ros2_control/HandRobotSystemPositionHardware</plugin>
             </hardware>
             <joint name="joint1">

Commit message: Fixing bugs. Include rviz config file. Able to work with view_robot.launch.py

File: description/ros2_control/handrobot.ros2_control.xacro (robot description, xacro)
@@ -1,6 +1,6 @@
 <?xml version="1.0"?>
-<robot xmlns:xacro="https://www.ros.org/wiki/xacro">
+<robot xmlns:xacro="http://www.ros.org/wiki/xacro">
     <xacro:macro name="handrobot_ros2_control" params="name">
-        <ros2_control name="${name}", type="system">
+        <ros2_control name="${name}" type="system">
             <hardware>
                 <plugin>handrobot_ros2_control/HandRobotSystemPositionHardware</plugin>

File: description/urdf/create_link.xacro (robot description, xacro)
@@ -2,10 +2,9 @@
 <robot xmlns:xacro="http://www.ros.org/wiki/xacro">
     <xacro:macro name="create_link" params="link_name xyz_offset rpy_offset mesh_package mesh_name color">
-    <xacro:include filename="$(find handrobot_ros2_control)/urdf/handrobot.materials.xacro" />
         <link name="${link_name}">
             <visual>
                 <origin xyz="${xyz_offset}" rpy="${rpy_offset}"/>
                 <geometry>
-                    <mesh filename="package://${mesh_package}/meshes/visual/${mesh_name}.stl" />
+                    <mesh filename="package://${mesh_package}/meshes/${mesh_name}.stl" scale="0.001 0.001 0.001"/>
                 </geometry>
                 <material name="${color}"/>
@@ -14,5 +13,5 @@
                 <origin xyz="${xyz_offset}" rpy="${rpy_offset}"/>
                 <geometry>
-                    <mesh filename="package://${mesh_package}/meshes/visual/${mesh_name}.stl" />
+                    <mesh filename="package://${mesh_package}/meshes/${mesh_name}.stl" scale="0.001 0.001 0.001"/>
                 </geometry>
             </collision>

File: description/urdf/handrobot.urdf.xacro (robot description, xacro)
@@ -1,4 +1,6 @@
 <?xml version="1.0"?>
-<robot xmlns:xacro="https://www.ros.org/wiki/xacro" name="HandRobot">
+<robot xmlns:xacro="http://www.ros.org/wiki/xacro" name="HandRobot">
+    <xacro:include filename="$(find handrobot_ros2_control)/urdf/handrobot.materials.xacro" />
+    <xacro:include filename="$(find handrobot_ros2_control)/urdf/create_link.xacro" />
     <xacro:include filename="$(find handrobot_ros2_control)/urdf/handrobot_description.urdf.xacro" />  <!-- Why is "description" not required before urdf...? -->
     <xacro:include filename="$(find handrobot_ros2_control)/ros2_control/handrobot.ros2_control.xacro" />

File: description/urdf/handrobot_description.urdf.xacro (robot description, xacro)
@@ -1,6 +1,5 @@
 <?xml version="1.0"?>
-<robot xmlns:xacro="https://www.ros.org/wiki/xacro">
+<robot xmlns:xacro="http://www.ros.org/wiki/xacro">
     <xacro:macro name="handrobot_description" params="parent *origin">
-    <xacro:include filename="$(find handrobot_ros2_control)/urdf/create_link.xacro" />
     <joint name="base_joint" type="fixed">
         <xacro:insert_block name="origin" />
@@ -10,5 +9,5 @@
     <xacro:create_link
         link_name="base_link"
-        xyz_offset="0 0 0"
+        xyz_offset="0 -0.025 0"
         rpy_offset="0 0 0"
         mesh_package="handrobot_ros2_control"
@@ -18,6 +17,6 @@
     <joint name="joint1" type="continuous">
         <parent link="base_link" />
-        <child link= "link1" />
-        <origin xyz="0 0.1 0" rpy="0 0 0"/>
+        <child link= "link_1" />
+        <origin xyz="0 0 0.1" rpy="0 0 0"/>
         <axis xyz="0 1 0"/>
         <dynamics damping="0.7"/>
@@ -26,5 +25,5 @@
     <xacro:create_link
         link_name="link_1"
-        xyz_offset="0 0 0"
+        xyz_offset="0 -0.02 0.0"
         rpy_offset="0 0 0"
         mesh_package="handrobot_ros2_control"

Commit message: Include five fingers descriptions!

File: description/ros2_control/handrobot.ros2_control.xacro (robot description, xacro)
@@ -13,4 +13,60 @@
                 <state_interface name="position"/>
             </joint>
+            <joint name="joint2-dm">
+                <command_interface name="position">
+                    <param name="min">-1</param>
+                    <param name="max">1</param>
+                </command_interface>
+                <state_interface name="position"/>
+            </joint>
+            <joint name="joint2-mu">
+                <command_interface name="position">
+                    <param name="min">-1</param>
+                    <param name="max">1</param>
+                </command_interface>
+                <state_interface name="position"/>
+            </joint>
+            <joint name="joint3-dm">
+                <command_interface name="position">
+                    <param name="min">-1</param>
+                    <param name="max">1</param>
+                </command_interface>
+                <state_interface name="position"/>
+            </joint>
+            <joint name="joint3-mu">
+                <command_interface name="position">
+                    <param name="min">-1</param>
+                    <param name="max">1</param>
+                </command_interface>
+                <state_interface name="position"/>
+            </joint>
+            <joint name="joint4-dm">
+                <command_interface name="position">
+                    <param name="min">-1</param>
+                    <param name="max">1</param>
+                </command_interface>
+                <state_interface name="position"/>
+            </joint>
+            <joint name="joint4-mu">
+                <command_interface name="position">
+                    <param name="min">-1</param>
+                    <param name="max">1</param>
+                </command_interface>
+                <state_interface name="position"/>
+            </joint>
+            <joint name="joint5-dm">
+                <command_interface name="position">
+                    <param name="min">-1</param>
+                    <param name="max">1</param>
+                </command_interface>
+                <state_interface name="position"/>
+            </joint>
+            <joint name="joint5-mu">
+                <command_interface name="position">
+                    <param name="min">-1</param>
+                    <param name="max">1</param>
+                </command_interface>
+                <state_interface name="position"/>
+            </joint>
         </ros2_control>
     </xacro:macro>

File: description/urdf/handrobot_description.urdf.xacro (robot description, xacro)
@@ -2,33 +2,218 @@
 <robot xmlns:xacro="http://www.ros.org/wiki/xacro">
     <xacro:macro name="handrobot_description" params="parent *origin">
-    <joint name="base_joint" type="fixed">
-        <xacro:insert_block name="origin" />
-        <parent link = "${parent}" />
-        <child link = "base_link" />
-    </joint>
-    <xacro:create_link
-        link_name="base_link"
-        xyz_offset="0 -0.025 0"
-        rpy_offset="0 0 0"
-        mesh_package="handrobot_ros2_control"
-        mesh_name="FirstPart"
-        color="blue"
+    <joint name="base_joint1" type="fixed">
+        <xacro:insert_block name="origin" />
+        <parent link = "${parent}" />
+        <child link = "one_down" />
+    </joint>
+    <joint name="base_joint2" type="fixed">
+        <xacro:insert_block name="origin" />
+        <parent link = "${parent}" />
+        <child link = "two_down" />
+    </joint>
+    <joint name="base_joint3" type="fixed">
+        <xacro:insert_block name="origin" />
+        <parent link = "${parent}" />
+        <child link = "three_down" />
+    </joint>
+    <joint name="base_joint4" type="fixed">
+        <xacro:insert_block name="origin" />
+        <parent link = "${parent}" />
+        <child link = "four_down" />
+    </joint>
+    <joint name="base_joint5" type="fixed">
+        <xacro:insert_block name="origin" />
+        <parent link = "${parent}" />
+        <child link = "five_down" />
+    </joint>
+    <!-- Joint 1 -->
+    <xacro:create_link
+        link_name="one_down"
+        xyz_offset="0 0 0"
+        rpy_offset="0 0 0"
+        mesh_package="handrobot_ros2_control"
+        mesh_name="OneDown"
+        color="blue"
+    />
+    <xacro:create_link
+        link_name="one_up"
+        xyz_offset="0 0 0.0"
+        rpy_offset="0 0 0"
+        mesh_package="handrobot_ros2_control"
+        mesh_name="OneUp"
+        color="orange"
     />
     <joint name="joint1" type="continuous">
-        <parent link="base_link" />
-        <child link= "link_1" />
-        <origin xyz="0 0 0.1" rpy="0 0 0"/>
-        <axis xyz="0 1 0"/>
-        <dynamics damping="0.7"/>
-        <limit effort="300" velocity="3.0"/>
-    </joint>
-    <xacro:create_link
-        link_name="link_1"
-        xyz_offset="0 -0.02 0.0"
-        rpy_offset="0 0 0"
-        mesh_package="handrobot_ros2_control"
-        mesh_name="SecondPart"
-        color="orange"
-    />
+        <parent link="one_down" />
+        <child link= "one_up" />
+        <origin xyz="0 0 0.035" rpy="0 0 0"/>
+        <axis xyz="0 1 0"/>
+        <dynamics damping="0.7"/>
+        <limit effort="300" velocity="3.0"/>
+    </joint>
+    <!-- Joint 2 -->
+    <xacro:create_link
+        link_name="two_down"
+        xyz_offset="0 0.04 0"
+        rpy_offset="0 0 0"
+        mesh_package="handrobot_ros2_control"
+        mesh_name="TwoDown"
+        color="blue"
+    />
+    <xacro:create_link
+        link_name="two_middle"
+        xyz_offset="0 0 0"
+        rpy_offset="0 0 0"
+        mesh_package="handrobot_ros2_control"
+        mesh_name="TwoMiddle"
+        color="green"
+    />
+    <xacro:create_link
+        link_name="two_up"
+        xyz_offset="0 0 0"
+        rpy_offset="0 0 0"
+        mesh_package="handrobot_ros2_control"
+        mesh_name="TwoUp"
+        color="orange"
+    />
+    <joint name="joint2-dm" type="continuous">
+        <parent link="two_down" />
+        <child link= "two_middle" />
+        <origin xyz="0 0.04 0.045" rpy="0 0 0"/>
+        <axis xyz="0 1 0"/>
+        <dynamics damping="0.7"/>
+        <limit effort="300" velocity="3.0"/>
+    </joint>
+    <joint name="joint2-mu" type="continuous">
+        <parent link="two_middle" />
+        <child link= "two_up" />
+        <origin xyz="0 0 0.025" rpy="0 0 0"/>
+        <axis xyz="0 1 0"/>
+        <dynamics damping="0.7"/>
+        <limit effort="300" velocity="3.0"/>
+    </joint>
+    <!-- Joint 3 -->
+    <xacro:create_link
+        link_name="three_down"
+        xyz_offset="0 0.08 0"
+        rpy_offset="0 0 0"
+        mesh_package="handrobot_ros2_control"
+        mesh_name="ThreeDown"
+        color="blue"
+    />
+    <xacro:create_link
+        link_name="three_middle"
+        xyz_offset="0 0 0"
+        rpy_offset="0 0 0"
+        mesh_package="handrobot_ros2_control"
+        mesh_name="ThreeMiddle"
+        color="green"
+    />
+    <xacro:create_link
+        link_name="three_up"
+        xyz_offset="0 0 0"
+        rpy_offset="0 0 0"
+        mesh_package="handrobot_ros2_control"
+        mesh_name="ThreeUp"
+        color="orange"
+    />
+    <joint name="joint3-dm" type="continuous">
+        <parent link="three_down" />
+        <child link= "three_middle" />
+        <origin xyz="0 0.08 0.05" rpy="0 0 0"/>
+        <axis xyz="0 1 0"/>
+        <dynamics damping="0.7"/>
+        <limit effort="300" velocity="3.0"/>
+    </joint>
+    <joint name="joint3-mu" type="continuous">
+        <parent link="three_middle" />
+        <child link= "three_up" />
+        <origin xyz="0 0 0.03" rpy="0 0 0"/>
+        <axis xyz="0 1 0"/>
+        <dynamics damping="0.7"/>
+        <limit effort="300" velocity="3.0"/>
+    </joint>
+    <!-- Joint 4 -->
+    <xacro:create_link
+        link_name="four_down"
+        xyz_offset="0 0.12 0"
+        rpy_offset="0 0 0"
+        mesh_package="handrobot_ros2_control"
+        mesh_name="FourDown"
+        color="blue"
+    />
+    <xacro:create_link
+        link_name="four_middle"
+        xyz_offset="0 0 0"
+        rpy_offset="0 0 0"
+        mesh_package="handrobot_ros2_control"
+        mesh_name="FourMiddle"
+        color="green"
+    />
+    <xacro:create_link
+        link_name="four_up"
+        xyz_offset="0 0 0"
+        rpy_offset="0 0 0"
+        mesh_package="handrobot_ros2_control"
+        mesh_name="FourUp"
+        color="orange"
+    />
+    <joint name="joint4-dm" type="continuous">
+        <parent link="four_down" />
+        <child link= "four_middle" />
+        <origin xyz="0 0.12 0.045" rpy="0 0 0"/>
+        <axis xyz="0 1 0"/>
+        <dynamics damping="0.7"/>
+        <limit effort="300" velocity="3.0"/>
+    </joint>
+    <joint name="joint4-mu" type="continuous">
+        <parent link="four_middle" />
+        <child link= "four_up" />
+        <origin xyz="0 0 0.03" rpy="0 0 0"/>
+        <axis xyz="0 1 0"/>
+        <dynamics damping="0.7"/>
+        <limit effort="300" velocity="3.0"/>
+    </joint>
+    <!-- Joint 5 -->
+    <xacro:create_link
+        link_name="five_down"
+        xyz_offset="0 0.16 0"
+        rpy_offset="0 0 0"
+        mesh_package="handrobot_ros2_control"
+        mesh_name="FiveDown"
+        color="blue"
+    />
+    <xacro:create_link
+        link_name="five_middle"
+        xyz_offset="0 0 0"
+        rpy_offset="0 0 0"
+        mesh_package="handrobot_ros2_control"
+        mesh_name="FiveMiddle"
+        color="green"
+    />
+    <xacro:create_link
+        link_name="five_up"
+        xyz_offset="0 0 0"
+        rpy_offset="0 0 0"
+        mesh_package="handrobot_ros2_control"
+        mesh_name="FiveUp"
+        color="orange"
+    />
+    <joint name="joint5-dm" type="continuous">
+        <parent link="five_down" />
+        <child link= "five_middle" />
+        <origin xyz="0 0.16 0.04" rpy="0 0 0"/>
+        <axis xyz="0 1 0"/>
+        <dynamics damping="0.7"/>
+        <limit effort="300" velocity="3.0"/>
+    </joint>
+    <joint name="joint5-mu" type="continuous">
+        <parent link="five_middle" />
+        <child link= "five_up" />
+        <origin xyz="0 0 0.02" rpy="0 0 0"/>
+        <axis xyz="0 1 0"/>
+        <dynamics damping="0.7"/>
+        <limit effort="300" velocity="3.0"/>
+    </joint>
     </xacro:macro>
 </robot>

Commit message: Better visualisation of the hand with a new part added.

File: description/ros2_control/handrobot.ros2_control.xacro (robot description, xacro)
@@ -6,5 +6,5 @@
                 <plugin>handrobot_ros2_control/HandRobotSystemPositionHardware</plugin>
             </hardware>
-            <joint name="joint1">
+            <joint name="joint1-du">
                 <command_interface name="position">
                     <param name="min">-1</param>

File: description/urdf/handrobot_description.urdf.xacro (robot description, xacro)
@@ -2,9 +2,17 @@
 <robot xmlns:xacro="http://www.ros.org/wiki/xacro">
     <xacro:macro name="handrobot_description" params="parent *origin">
-    <joint name="base_joint1" type="fixed">
-        <xacro:insert_block name="origin" />
-        <parent link = "${parent}" />
-        <child link = "one_down" />
-    </joint>
+    <joint name="base_joint" type="fixed">
+        <xacro:insert_block name="origin" />
+        <parent link = "${parent}" />
+        <child link = "base" />
+    </joint>
+    <xacro:create_link
+        link_name="base"
+        xyz_offset="0 0 0"
+        rpy_offset="0 0 0"
+        mesh_package="handrobot_ros2_control"
+        mesh_name="Base"
+        color="yellow"
+    />
     <joint name="base_joint2" type="fixed">
         <xacro:insert_block name="origin" />
@@ -44,5 +52,10 @@
         color="orange"
     />
-    <joint name="joint1" type="continuous">
+    <joint name="joint1-bd" type="fixed">
+        <parent link="base" />
+        <child link= "one_down" />
+        <origin xyz="0 -0.055 0.035" rpy="0.7854 0 0"/>
+    </joint>
+    <joint name="joint1-du" type="continuous">
         <parent link="one_down" />
         <child link= "one_up" />
@@ -55,5 +68,5 @@
     <xacro:create_link
         link_name="two_down"
-        xyz_offset="0 0.04 0"
+        xyz_offset="0 -0.02 0"
         rpy_offset="0 0 0"
         mesh_package="handrobot_ros2_control"
@@ -77,8 +90,13 @@
         color="orange"
     />
+    <joint name="joint2-bd" type="fixed">
+        <parent link="base" />
+        <child link= "two_down" />
+        <origin xyz="0 -0.005 0.095" rpy="0.2618 0 0"/>
+    </joint>
     <joint name="joint2-dm" type="continuous">
         <parent link="two_down" />
         <child link= "two_middle" />
-        <origin xyz="0 0.04 0.045" rpy="0 0 0"/>
+        <origin xyz="0 -0.02 0.045" rpy="0 0 0"/>
         <axis xyz="0 1 0"/>
         <dynamics damping="0.7"/>
@@ -96,5 +114,5 @@
     <xacro:create_link
         link_name="three_down"
-        xyz_offset="0 0.08 0"
+        xyz_offset="0 0 0"
         rpy_offset="0 0 0"
         mesh_package="handrobot_ros2_control"
@@ -118,8 +136,13 @@
         color="orange"
     />
+    <joint name="joint3-bd" type="fixed">
+        <parent link="base" />
+        <child link= "three_down" />
+        <origin xyz="0 0 0.1" rpy="0 0 0"/>
+    </joint>
     <joint name="joint3-dm" type="continuous">
         <parent link="three_down" />
         <child link= "three_middle" />
-        <origin xyz="0 0.08 0.05" rpy="0 0 0"/>
+        <origin xyz="0 0 0.05" rpy="0 0 0"/>
         <axis xyz="0 1 0"/>
         <dynamics damping="0.7"/>
@@ -137,5 +160,5 @@
     <xacro:create_link
         link_name="four_down"
-        xyz_offset="0 0.12 0"
+        xyz_offset="0 0 0"
         rpy_offset="0 0 0"
         mesh_package="handrobot_ros2_control"
@@ -159,8 +182,13 @@
         color="orange"
     />
+    <joint name="joint4-bd" type="fixed">
+        <parent link="base" />
+        <child link= "four_down" />
+        <origin xyz="0 0.025 0.095" rpy="-0.2618 0 0"/>
+    </joint>
     <joint name="joint4-dm" type="continuous">
         <parent link="four_down" />
         <child link= "four_middle" />
-        <origin xyz="0 0.12 0.045" rpy="0 0 0"/>
+        <origin xyz="0 0 0.045" rpy="0 0 0"/>
         <axis xyz="0 1 0"/>
         <dynamics damping="0.7"/>
@@ -178,5 +206,5 @@
     <xacro:create_link
         link_name="five_down"
-        xyz_offset="0 0.16 0"
+        xyz_offset="0 0 0"
         rpy_offset="0 0 0"
         mesh_package="handrobot_ros2_control"
@@ -200,8 +228,13 @@
         color="orange"
     />
+    <joint name="joint5-bd" type="fixed">
+        <parent link="base" />
+        <child link= "five_down" />
+        <origin xyz="0 0.045 0.085" rpy="-0.524 0 0"/>
+    </joint>
     <joint name="joint5-dm" type="continuous">
         <parent link="five_down" />
         <child link= "five_middle" />
-        <origin xyz="0 0.16 0.04" rpy="0 0 0"/>
+        <origin xyz="0 0 0.04" rpy="0 0 0"/>
         <axis xyz="0 1 0"/>
         <dynamics damping="0.7"/>
