Commit message: Include other joints control in ControllerManager, URDF files, and camera control node.

File: description/ros2_control/handrobot.ros2_control.xacro (robot description, xacro)
@@ -6,5 +6,21 @@
                 <plugin>handrobot_ros2_control/HandRobotSystemPositionHardware</plugin>
             </hardware>
+            <!-- Joint 1 -->
+            <joint name="joint1-bd">
+                <command_interface name="position">
+                    <param name="min">-1</param>
+                    <param name="max">1</param>
+                </command_interface>
+                <state_interface name="position"/>
+            </joint>
             <joint name="joint1-du">
+                <command_interface name="position">
+                    <param name="min">-1</param>
+                    <param name="max">1</param>
+                </command_interface>
+                <state_interface name="position"/>
+            </joint>
+            <!-- Joint 2 -->
+            <joint name="joint2-bd">
                 <command_interface name="position">
                     <param name="min">-1</param>
@@ -27,4 +43,12 @@
                 <state_interface name="position"/>
             </joint>
+            <!-- Joint 3 -->
+            <joint name="joint3-bd">
+                <command_interface name="position">
+                    <param name="min">-1</param>
+                    <param name="max">1</param>
+                </command_interface>
+                <state_interface name="position"/>
+            </joint>
             <joint name="joint3-dm">
                 <command_interface name="position">
@@ -41,4 +65,12 @@
                 <state_interface name="position"/>
             </joint>
+            <!-- Joint 4 -->
+            <joint name="joint4-bd">
+                <command_interface name="position">
+                    <param name="min">-1</param>
+                    <param name="max">1</param>
+                </command_interface>
+                <state_interface name="position"/>
+            </joint>
             <joint name="joint4-dm">
                 <command_interface name="position">
@@ -49,4 +81,12 @@
             </joint>
             <joint name="joint4-mu">
+                <command_interface name="position">
+                    <param name="min">-1</param>
+                    <param name="max">1</param>
+                </command_interface>
+                <state_interface name="position"/>
+            </joint>
+            <!-- Joint 5 -->
+            <joint name="joint5-bd">
                 <command_interface name="position">
                     <param name="min">-1</param>

File: description/urdf/handrobot_description.urdf.xacro (robot description, xacro)
@@ -32,8 +32,11 @@
         color="orange"
     />
-    <joint name="joint1-bd" type="fixed">
+    <joint name="joint1-bd" type="continuous">
         <parent link="base" />
         <child link= "one_down" />
         <origin xyz="0 -0.055 0.035" rpy="0.7854 0 0"/>
+        <axis xyz="0 1 0"/>
+        <dynamics damping="0.7"/>
+        <limit effort="300" velocity="3.0"/>
     </joint>
     <joint name="joint1-du" type="continuous">
@@ -70,8 +73,11 @@
         color="orange"
     />
-    <joint name="joint2-bd" type="fixed">
+    <joint name="joint2-bd" type="continuous">
         <parent link="base" />
         <child link= "two_down" />
         <origin xyz="0 -0.005 0.095" rpy="0.2618 0 0"/>
+        <axis xyz="0 1 0"/>
+        <dynamics damping="0.7"/>
+        <limit effort="300" velocity="3.0"/>
     </joint>
     <joint name="joint2-dm" type="continuous">
@@ -116,8 +122,11 @@
         color="orange"
     />
-    <joint name="joint3-bd" type="fixed">
+    <joint name="joint3-bd" type="continuous">
         <parent link="base" />
         <child link= "three_down" />
         <origin xyz="0 0 0.1" rpy="0 0 0"/>
+        <axis xyz="0 1 0"/>
+        <dynamics damping="0.7"/>
+        <limit effort="300" velocity="3.0"/>
     </joint>
     <joint name="joint3-dm" type="continuous">
@@ -162,8 +171,11 @@
         color="orange"
     />
-    <joint name="joint4-bd" type="fixed">
+    <joint name="joint4-bd" type="continuous">
         <parent link="base" />
         <child link= "four_down" />
         <origin xyz="0 0.025 0.095" rpy="-0.2618 0 0"/>
+        <axis xyz="0 1 0"/>
+        <dynamics damping="0.7"/>
+        <limit effort="300" velocity="3.0"/>
     </joint>
     <joint name="joint4-dm" type="continuous">
@@ -208,8 +220,11 @@
         color="orange"
     />
-    <joint name="joint5-bd" type="fixed">
+    <joint name="joint5-bd" type="continuous">
         <parent link="base" />
         <child link= "five_down" />
         <origin xyz="0 0.045 0.085" rpy="-0.524 0 0"/>
+        <axis xyz="0 1 0"/>
+        <dynamics damping="0.7"/>
+        <limit effort="300" velocity="3.0"/>
     </joint>
     <joint name="joint5-dm" type="continuous">
